Commit message: fix rotation
Signed-off-by: wam-v-tan <ouxt.share@gmail.com>

File: config/urdf/miniv_sensors.urdf (robot description, URDF)
Before this commit: robot miniv_sensors, 4 links, 3 joints
Joints:
- joint front_base_link_to_velodyne_joint: origin xyz=0.2 0 0.1 rpy=0 0 0 -> xyz=0.2 0 0.1 rpy=3.141592653589793 0 0
- joint front_velodyne_to_camera_joint: origin xyz=0 0 0 rpy=0 0 0 -> xyz=0 0 0 rpy=3.141592653589793 0 0

Commit message: configure sensor
Signed-off-by: wam-v-tan <ouxt.share@gmail.com>

File: config/urdf/miniv_sensors.urdf (robot description, URDF)
Before this commit: robot miniv_sensors, 4 links, 3 joints
Joints:
- joint front_velodyne_to_camera_joint: origin xyz=0 0 0 rpy=3.141592653589793 0 0 -> xyz=0.03 0 0 rpy=3.141592653589793 0 0

Commit message: update parameter
Signed-off-by: wam-v-tan <ouxt.share@gmail.com>

File: config/urdf/miniv_sensors.urdf (robot description, URDF)
Before this commit: robot miniv_sensors, 4 links, 3 joints
Joints:
- joint front_velodyne_to_camera_joint: origin xyz=0.03 0 0 rpy=3.141592653589793 0 0 -> xyz=0.05 0 -0.08 rpy=3.141592653589793 0 0
